Commit message: working sim launch file

File: install/uorover_arm/share/uorover_arm/urdf/rmm.urdf (robot description, URDF)
Before this commit: robot rmm, 6 links, 5 joints
Joints:
- joint q4: origin xyz=0.25 0 0.00014259 rpy=0 0 0.3938 -> xyz=0.25 0 0.0014259 rpy=0 0 0

File: install/uorover_moveit_config/share/uorover_moveit_config/config/rmm.urdf.xacro (robot description, xacro)
@@ -1,8 +1,10 @@
 <?xml version="1.0"?>
 <robot xmlns:xacro="http://www.ros.org/wiki/xacro" name="rmm">
-    <xacro:arg name="initial_positions_file" default="initial_positions.yaml" />
+    <xacro:arg name="use_mock_hardware" default="false" />
     <xacro:include filename="$(find uorover_arm)/urdf/rmm.urdf" />
     <!-- Import control_xacro -->
     <xacro:include filename="rmm_ros2_control.xacro" />
-    <xacro:rmm_ros2_control name="ArmSystem" initial_positions_file="$(arg initial_positions_file)"/>
+    <xacro:rmm_ros2_control
+     	name="ArmSystem"
+     	use_mock_hardware="$(arg use_mock_hardware)" />
 </robot>

File: install/uorover_moveit_config/share/uorover_moveit_config/config/rmm_ros2_control.xacro (robot description, xacro)
@@ -1,14 +1,18 @@
 <?xml version="1.0"?>
 <robot xmlns:xacro="http://www.ros.org/wiki/xacro">
-    <xacro:macro name="rmm_ros2_control" params="name initial_positions_file">
-        <xacro:property name="initial_positions" value="${load_yaml(initial_positions_file)['initial_positions']}"/>
+    <xacro:macro name="rmm_ros2_control" params="name use_mock_hardware:=^|true">
         <ros2_control name="${name}" type="system">
             <hardware>
-                <plugin>uorover_ik/ArmSystem</plugin>
+            	<xacro:if value="${use_mock_hardware}">
+            		<plugin>mock_components/GenericSystem</plugin>
+            	</xacro:if>
+            	<xacro:unless value="${use_mock_hardware}">
+            		<plugin>uorover_ik/ArmSystem</plugin>
+            	</xacro:unless>
             </hardware>
             <joint name="q1">
                 <command_interface name="position"/>
                 <state_interface name="position">
-                  <param name="initial_value">${initial_positions['q1']}</param>
+                <param name="initial_value">0.0</param>
                 </state_interface>
                 <state_interface name="velocity"/>
@@ -17,5 +21,5 @@
                 <command_interface name="position"/>
                 <state_interface name="position">
-                  <param name="initial_value">${initial_positions['q2']}</param>
+                  <param name="initial_value">0.0</param>
                 </state_interface>
                 <state_interface name="velocity"/>
@@ -24,5 +28,5 @@
                 <command_interface name="position"/>
                 <state_interface name="position">
-                  <param name="initial_value">${initial_positions['q3']}</param>
+                  <param name="initial_value">1.3439</param>
                 </state_interface>
                 <state_interface name="velocity"/>
@@ -31,5 +35,5 @@
                 <command_interface name="position"/>
                 <state_interface name="position">
-                  <param name="initial_value">${initial_positions['q4']}</param>
+                  <param name="initial_value">0</param>
                 </state_interface>
                 <state_interface name="velocity"/>
